File: Schematics + Pcb/Power_stage.kicad_sch (KiCad schematic)
At the start: 12 parts

Commit message: Work in progress
Parts:
- removed C?: 10uF, symbol Device:C_Polarized_Small
- removed D?: 60V, symbol Device:D_Schottky
- removed FB? (x2): FerriteBead, symbol Device:FerriteBead_Small
- removed IC?: MIC4605-2YMT-TR, SON50P250X250X60-11N-D, symbol MIC4605-2YMT-TR:MIC4605-2YMT-TR
- added D?: 15V, symbol Device:D_Schottky
- added IC?: STGAP2HDMTR, STGAP2HDMTR, symbol STGAP2HDMTR:STGAP2HDMTR
- added PS?: PDSE1-S12-S3-D, PDSE1S12S3D, symbol PDSE1-S12-S3-D:PDSE1-S12-S3-D
- added R? (x4): R, symbol Device:R
- added R? (x4): (no value), symbol Device:R
- added U? (x2): WYBRAĆ!, Package_DIP:SMDIP-4_W9.53mm_Clearance8mm, symbol Isolator:SFH617A-3X017T
- added U?: Current sense amplifier, symbol pspice:OPAMP
Connections:
- net OUTPUT is gone; now on net +12V: 220uH?.2, C?.1, C?.1, C?.1
- net +12V: now also D?.1 (K), PS?.4 (VIN), R?.1, U?.4 (V+)
- net GND: now also PS?.7 (0V), U?.3, U?.3; no longer C?.2, C?.2, C?.2, Q?.3 (S)
- net HS: now also R?.2
- net Vdrive: now reaches Q?.1 (D)
- net SENSE+: now reaches Q?.3 (S), R1-Sense?.1
- net SENSE+: now also R?.1
- new net: R?.2, U?.1 (x2)
- new net: R?.1, R?.2, U?.1 (+)
- new net: R?.1, R?.2, U?.2 (-)
- new net: R?.1, R?.1, U?.3
- new net +3V3: PS?.5 (+VOUT), R?.1, R?.1
- new net Current sense output: R?.2, U?.4
- new net GNDPWR: C?.2, C?.2, C?.2, D?.2 (A), PS?.1 (GND), Q?.3 (S), R?.2, U?.2, U?.2, U?.5 (V-)
- new net Voltage measure point : R?.2, U?.4
- no-connect marks 2 -> 0
Other:
- note added: "Może zamiast pół-mostka dać flyback dla izolacji."
- moved on the sheet: 220uH?, C?, Q?, R1-Sense?
