File: Schematics + Pcb/Praca_Inżynierska.kicad_sch (KiCad schematic)
At the start: 31 parts

Commit message: Added function diagram
Parts:
- removed C? (x2): 10u, symbol Device:C_Polarized_Small
- removed C?: C_Delay, symbol Device:C_Small
- removed C? (x2): 1u, symbol Device:C_Polarized_Small
- removed C?: 10uF, symbol Device:C
- removed D?: SD05_SOD323, Diode_SMD:D_SOD-323, symbol Diode:SD05_SOD323
- removed FB?: FerriteBead_OUTPUT, symbol Device:FerriteBead_Small
- removed FB?: FerriteBead_INPUT, symbol Device:FerriteBead_Small
- removed IC?: NCV8501D50R2G, SOIC127P600X175-8N, symbol NCV8501D50R2G:NCV8501D50R2G
- removed IC?: S-1212BC0-M5T1U, SOT95P275X130-5N, symbol S-1212BC0-M5T1U:S-1212BC0-M5T1U
- removed R? (x2): R, symbol Device:R
- removed R? (x2): 10k, symbol Device:R
- removed R?: 100k, symbol Device:R
- removed U?: ADG419BN, Package_DIP:DIP-8_W7.62mm, symbol Analog_Switch:ADG419BN
Other:
- removed sheet StandaloneSheet
- added sheet Standby_power (Coincell.kicad_sch)
- note added: "Co dodać: ~Sterownik półmostka -Stabilizator liniowy 5V -USB -skalowanie napięcia dla mikrokontrolera -Voltage Feedback -Current Sensing -Diody stanu -Connectory"
- note added: "Microcontroller Power z coina"
- note added: "Może pamięć z parametrami?"
- note added: "zmodyfikować"
- note removed: "-Start logiki z coina"
- note removed: "Bridge Driver Power"
- note removed: "Co dodać: ~Sterownik półmostka -Stabilizator liniowy 5V -USB -skalowanie napięcia dla mikrokontrolera -Voltage Feedback -Current Sensing -Diody stanu -Przełącznik do StandAlone -potencjometry do StandAlone -Connectory -USB C do ładowania telefonu"
- note removed: "Microcontroller Power"
- note removed: "Reference voltage zamiast Dzielnika napięcia na MONITOR! Sprawdzić w doksach atmegi minimalne napięcie pracy!"
- note removed: "Sprawdzić"
- note removed: "Standalone Mode"
- note removed: "Zmienić napięcie zasialnia na większe niż 5V"
- moved on the sheet: C?, Y?

Commit message: Work in progress
Parts:
- removed C?: 0.1uF, symbol Device:C
- removed U?: ATmega328-P, Package_DIP:DIP-28_W7.62mm, symbol MCU_Microchip_ATmega:ATmega328-P
- added C?: 10uF, symbol Device:C_Small
- added FB?: FerriteBead_Small, symbol Device:FerriteBead_Small
- added IC?: STM32L4P5RET6, QFP50P1200X1200X160-64N, symbol STM32L4P5RET6:STM32L4P5RET6
- added R?: 100k, symbol Device:R
- added SW?: Reset Switch, symbol Switch:SW_MEC_5G
- C? (x2): value 33pF -> 22pF
Connections:
- net GND: now also C?.2, IC?.12 (VSSA/VREF-), IC?.18 (VSS_1), IC?.31 (VSS_2), IC?.47 (VSS_3), IC?.63 (VSS_4), R?.2
- net XTAL1: now also C?.1, Y?.1, IC?.5 (PH0-OSC_IN); no longer C?.1, Y?.2
- net XTAL2: now also C?.1, Y?.2, IC?.6 (PH1-OSC_OUT); no longer C?.1, Y?.1
- net ~{RESET}: now also R?.1, SW?.3 (B), SW?.4 (B)
- net +5V: no longer names the net of C?.1, C?.1, C?.1
- net +5V: now also C?.1, FB?.2
- new net +3V3: FB?.1, IC?.13 (VDDA/VREF+), IC?.19 (VDD_1), IC?.32 (VDD_2), IC?.64 (VDD_3), SW?.1 (A), SW?.2 (A)
- no-connect marks 1 -> 0
Other:
- removed sheet Current_Sense
- removed sheet USB
- removed sheet Voltage_Feedback
- removed sheet Voltage_Probing
- added sheet Middle stage (Middle_Stage.kicad_sch)
- note added: "Connectors + USB"
- note added: "MIDDLE STAGE"
- note added: "OUTPUT STAGE"
- note removed: "Co dodać: ~Sterownik półmostka -Stabilizator liniowy 5V -USB -skalowanie napięcia dla mikrokontrolera -Voltage Feedback -Current Sensing -Diody stanu -Connectory"
- note removed: "Connectors"
- note removed: "Current sense"
- note removed: "Może pamięć z parametrami?"
- note removed: "Power"
- note removed: "USB"
- note removed: "Voltage Feedback"
- note removed: "Voltage Probing"
- note removed: "Zrobić"
- note removed: "zmodyfikować"
- moved on the sheet: C?, Y?
