File: Schematics + Pcb/USB.kicad_sch (KiCad schematic)
At the start: 0 parts

Commit message: Work in progress
Parts:
- added J?: (no value), symbol Connector:USB_B_Micro
- added R? (x2): (no value), symbol Device:R
Connections:
- new net: J?.2 (D-), R?.1
- new net: J?.3 (D+), R?.1
- new net +5V: J?.1 (VBUS)
- new net GND: J?.5 (GND)
- no-connect marks 0 -> 2
Changed lines of the file:
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@@
 (kicad_sch (version 20211123) (generator eeschema)
   (paper "A4")
+  (no_connect (at 61.595 52.07))
+  (no_connect (at 51.435 57.15))
+  (wire (pts (xy 61.595 41.91) (xy 63.5 41.91))
+    (stroke (width 0) (type default) (color 0 0 0 0))
+  )
+  (wire (pts (xy 61.595 46.99) (xy 64.135 46.99))
+    (stroke (width 0) (type default) (color 0 0 0 0))
+  )
+  (wire (pts (xy 61.595 49.53) (xy 64.135 49.53))
+    (stroke (width 0) (type default) (color 0 0 0 0))
+  )
+  (wire (pts (xy 63.5 38.735) (xy 63.5 41.91))
+    (stroke (width 0) (type default) (color 0 0 0 0))
+  )
+  (wire (pts (xy 53.975 59.055) (xy 53.975 57.15))
+    (stroke (width 0) (type default) (color 0 0 0 0))
+  )
+  (symbol (lib_id "Connector:USB_B_Micro") (at 53.975 46.99 0) (unit 1)
+    (in_bom yes) (on_board yes) (fields_autoplaced)
+    (property "Reference" "J?" (id 0) (at 53.975 34.29 0))
+    (property "Value" "" (id 1) (at 53.975 36.83 0))
+    (property "Footprint" "" (id 2) (at 57.785 48.26 0)
+      (effects (font (size 1.27 1.27)) hide)
+    )
+    (property "Datasheet" "~" (id 3) (at 57.785 48.26 0)
+      (effects (font (size 1.27 1.27)) hide)
+    )
+    (pin "1")
+    (pin "2")
+    (pin "3")
+    (pin "4")
+    (pin "5")
+    (pin "6")
+  )
+  (symbol (lib_id "power:GND") (at 53.975 59.055 0) (unit 1)
+    (in_bom yes) (on_board yes) (fields_autoplaced)
+    (property "Reference" "#PWR?" (id 0) (at 53.975 65.405 0)
+      (effects (font (size 1.27 1.27)) hide)
+    )
+    (property "Value" "" (id 1) (at 53.975 64.135 0))
+    (property "Footprint" "" (id 2) (at 53.975 59.055 0)
+      (effects (font (size 1.27 1.27)) hide)
+    )
+    (property "Datasheet" "" (id 3) (at 53.975 59.055 0)
+      (effects (font (size 1.27 1.27)) hide)
+    )
+    (pin "1")
+  )
+  (symbol (lib_id "power:+5V") (at 63.5 38.735 0) (unit 1)
+    (in_bom yes) (on_board yes)
+    (property "Reference" "#PWR?" (id 0) (at 63.5 42.545 0)
+      (effects (font (size 1.27 1.27)) hide)
+    )
+    (property "Value" "" (id 1) (at 63.5 35.179 0))
+    (property "Footprint" "" (id 2) (at 63.5 38.735 0)
+      (effects (font (size 1.27 1.27)) hide)
+    )
+    (property "Datasheet" "" (id 3) (at 63.5 38.735 0)
+      (effects (font (size 1.27 1.27)) hide)
+    )
+    (pin "1")
+  )
+  (symbol (lib_id "Device:R") (at 67.945 49.53 90) (unit 1)
+    (in_bom yes) (on_board yes)
+    (property "Reference" "R?" (id 0) (at 66.675 53.975 90))
+    (property "Value" "" (id 1) (at 66.04 52.07 90))
+    (property "Footprint" "" (id 2) (at 67.945 51.308 90)
+      (effects (font (size 1.27 1.27)) hide)
+    )
+    (property "Datasheet" "~" (id 3) (at 67.945 49.53 0)
+      (effects (font (size 1.27 1.27)) hide)
+    )
+    (pin "1")
+    (pin "2")
+  )
+  (symbol (lib_id "Device:R") (at 67.945 46.99 90) (unit 1)
+    (in_bom yes) (on_board yes)
+    (property "Reference" "R?" (id 0) (at 66.675 43.18 90))
+    (property "Value" "" (id 1) (at 66.04 45.085 90))
+    (property "Footprint" "" (id 2) (at 67.945 48.768 90)
+      (effects (font (size 1.27 1.27)) hide)
+    )
+    (property "Datasheet" "~" (id 3) (at 67.945 46.99 0)
+      (effects (font (size 1.27 1.27)) hide)
+    )
+    (pin "1")
+    (pin "2")
+  )
 )
